Commit message: Included two worlds and Readme updated

File: urdf/warthog_velodyne.urdf.xacro (robot description, xacro)
@@ -335,5 +335,5 @@
   <joint name="camera_joint" type="fixed">
     <axis xyz="0 0 0" />
-    <origin xyz="${(chassis_length / 2) - (camera_box / 2) - 0.02} 0 ${chassis_height + (camera_box / 2) - 0.01}" rpy="0 0 0"/>
+    <origin xyz="${(chassis_length / 2) - (camera_box / 2) - 0.02 + 0.1} 0 ${chassis_height + (camera_box / 2) - 0.01}" rpy="0 3.141592654 3.141592654"/>
     <parent link="base_link"/>
     <child link="camera_link"/>
@@ -341,5 +341,5 @@
   <link name="camera_link">
     <collision>
-      <origin xyz="0 0 10" rpy="0 0 0"/>
+      <origin xyz="0 0 0" rpy="0 0 0"/>
       <geometry>
     <box size="${camera_box / 2} ${camera_box} ${camera_box}"/>
@@ -369,6 +369,6 @@
         <horizontal_fov>1.4</horizontal_fov>
         <image>
-          <width>800</width>
-          <height>800</height>
+          <width>1280</width>
+          <height>720</height>
           <format>R8G8B8</format>
         </image>
